File: hw/ipibitsy.kicad_pcb (KiCad board)
At the start: 2 copper layers, 100 x 100 mm, 176 parts, among them J101 Conn_02x25_Odd_Even, J102 Barrel_Jack_Switch, U1001 SN75176AD, U101 YAAJ_WeAct_BlackPill_Part_Lik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, U102 MP1584EN_MOD, U1101 SN75176AD, U1201 SN75176AD, U1301 SN75176AD, U1401 SN75176AD, U1501 SN75176AD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

Commit message: BUS*B* Parity bit driver direction pin was accidentally connected to BUS*A* direction net
Connections:
- U2001 pad 2: /Line Drivers/BUS_A.DIR -> /Line Drivers/BUS_B.DIR
- U2001 pad 3: /Line Drivers/BUS_A.DIR -> /Line Drivers/BUS_B.DIR
Routing:
- net /Line Drivers/BUS_A.DIR: track 317.7 -> 292.4 mm
- net /Line Drivers/BUS_B.DIR: track 302.3 -> 314.3 mm, vias 20 -> 21
