File: hw/trx_drv.kicad_sch (KiCad schematic)
At the start: 7 parts, among them U2001 SN75176AD

Commit message: BUS*B* Parity bit driver direction pin was accidentally connected to BUS*A* direction net
Parts:
- renumbered C1101 to C801, R2001 to R801, R1102 to R802, R1103 to R803, R2004 to R804, R2005 to R805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
